File: pcb_v2/pcb/pcb.kicad_pcb (KiCad board)
At the start: 2 copper layers, 104.2 x 99.5 mm, 28 parts, among them J1 Screw_Terminal_01x02, J2 Screw_Terminal_01x04, J3 Screw_Terminal_01x04, Q1 2N7000, Q2 2N7000, Q3 2N7000

Commit message: final report
Connections:
- D1 pad 1: +12V -> Net-(D1-K)
- D1 pad 2: GND -> +12V
- PTCFuse1 pad 1: +12V -> Net-(D1-K)
Routing:
- net Net-(D1-K): track 0.00 -> 7.65 mm
Changed lines of the file:
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@@
 	(net 58 "/EN_water")
 	(net 59 "/M0_water")
+	(net 60 "Net-(D1-K)")
 	(footprint "Capacitor_SMD:C_0805_2012Metric_Pad1.18x1.45mm_HandSolder"
 		(layer "F.Cu")
@@
 			(layers "F.Cu" "F.Mask" "F.Paste")
 			(roundrect_rratio 0.175439)
-			(net 49 "+12V")
+			(net 60 "Net-(D1-K)")
 			(pintype "passive")
 		)
@@
 			(layers "*.Cu" "*.Mask")
 			(remove_unused_layers no)
-			(net 49 "+12V")
+			(net 60 "Net-(D1-K)")
 			(pinfunction "K")
 			(pintype "passive")
@@
 			(layers "*.Cu" "*.Mask")
 			(remove_unused_layers no)
-			(net 23 "GND")
+			(net 49 "+12V")
 			(pinfunction "A")
 			(pintype "passive")
@@
 		(net 59)
 	)
+	(segment
+		(start 122.42 139)
+		(end 122.42 144.42)
+		(width 0.3)
+		(layer "B.Cu")
+		(net 60)
+	)
+	(segment
+		(start 122.42 144.42)
+		(end 124 146)
+		(width 0.3)
+		(layer "B.Cu")
+		(net 60)
+	)
 	(zone
