File: pcb_v2/pcb/pcb.kicad_sch (KiCad schematic)
At the start: 28 parts, among them J1 Screw_Terminal_01x02, J2 Screw_Terminal_01x04, J3 Screw_Terminal_01x04, Q1 2N7000, Q2 2N7000, Q3 2N7000

Commit message: final report
Connections:
- net +12V: now also D1.2 (A); no longer D1.1 (K), PTCFuse1.1
- net GND: no longer D1.2 (A)
- new net: D1.1 (K), PTCFuse1.1
Other:
- moved on the sheet: D1
Changed lines of the file:
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@@
 	)
 	(junction
+		(at 181.61 33.02)
+		(diameter 0)
+		(color 0 0 0 0)
+	)
+	(junction
 		(at 146.05 127)
 		(diameter 0)
@@
 	)
 	(junction
-		(at 172.72 24.13)
-		(diameter 0)
-		(color 0 0 0 0)
-	)
-	(junction
 		(at 154.94 33.02)
 		(diameter 0)
@@
 	)
 	(junction
-		(at 181.61 33.02)
-		(diameter 0)
-		(color 0 0 0 0)
-	)
-	(junction
 		(at 67.31 50.8)
 		(diameter 0)
@@
 	)
 	(junction
-		(at 172.72 33.02)
-		(diameter 0)
-		(color 0 0 0 0)
-	)
-	(junction
 		(at 191.77 24.13)
 		(diameter 0)
@@
 	(wire
 		(pts
+			(xy 172.72 33.02) (xy 173.99 33.02)
+		)
+		(stroke
+			(width 0)
+			(type default)
+		)
+	)
+	(wire
+		(pts
 			(xy 229.87 124.46) (xy 276.86 124.46)
 		)
@@
 	(wire
 		(pts
-			(xy 172.72 24.13) (xy 186.69 24.13)
-		)
-		(stroke
-			(width 0)
-			(type default)
-		)
-	)
-	(wire
-		(pts
 			(xy 217.17 121.92) (xy 132.08 121.92)
 		)
@@
 	(wire
 		(pts
-			(xy 133.35 49.53) (xy 181.61 49.53)
+			(xy 133.35 48.26) (xy 181.61 48.26)
 		)
 		(stroke
@@
 	(wire
 		(pts
-			(xy 154.94 24.13) (xy 172.72 24.13)
-		)
-		(stroke
-			(width 0)
-			(type default)
-		)
-	)
-	(wire
-		(pts
 			(xy 66.04 71.12) (xy 66.04 80.01)
 		)
@@
 	(wire
 		(pts
+			(xy 154.94 24.13) (xy 186.69 24.13)
+		)
+		(stroke
+			(width 0)
+			(type default)
+		)
+	)
+	(wire
+		(pts
 			(xy 123.19 44.45) (xy 135.89 44.45)
 		)
@@
 	(wire
 		(pts
-			(xy 172.72 33.02) (xy 181.61 33.02)
-		)
-		(stroke
-			(width 0)
-			(type default)
-		)
-	)
-	(wire
-		(pts
 			(xy 237.49 101.6) (xy 241.3 101.6)
 		)
@@
 	(wire
 		(pts
-			(xy 172.72 31.75) (xy 172.72 33.02)
-		)
-		(stroke
-			(width 0)
-			(type default)
-		)
-	)
-	(wire
-		(pts
 			(xy 106.68 45.72) (xy 121.92 45.72)
 		)
@@
 	(wire
 		(pts
-			(xy 181.61 49.53) (xy 181.61 33.02)
+			(xy 181.61 48.26) (xy 181.61 33.02)
 		)
 		(stroke
@@
 	(wire
 		(pts
-			(xy 133.35 67.31) (xy 133.35 49.53)
+			(xy 133.35 67.31) (xy 133.35 48.26)
 		)
 		(stroke
@@
 	(symbol
 		(lib_id "Diode:1N4001")
-		(at 172.72 27.94 90)
+		(at 177.8 33.02 0)
 		(unit 1)
 		(exclude_from_sim no)
@@
 		(fields_autoplaced yes)
 		(property "Reference" "D1"
-			(at 175.26 26.6699 90)
+			(at 177.8 26.67 0)
 			(effects
 				(font
 					(size 1.27 1.27)
 				)
-				(justify right)
 			)
 		)
 		(property "Value" "1N4001"
-			(at 175.26 29.2099 90)
+			(at 177.8 29.21 0)
 			(effects
 				(font
 					(size 1.27 1.27)
 				)
-				(justify right)
 			)
 		)
 		(property "Footprint" "Diode_THT:D_DO-41_SOD81_P10.16mm_Horizontal"
-			(at 172.72 27.94 0)
+			(at 177.8 33.02 0)
 			(effects
 				(font
@@
 		)
 		(property "Datasheet" "http://www.vishay.com/docs/88503/1n4001.pdf"
-			(at 172.72 27.94 0)
+			(at 177.8 33.02 0)
 			(effects
 				(font
@@
 		)
 		(property "Description" "50V 1A General Purpose Rectifier Diode, DO-41"
-			(at 172.72 27.94 0)
+			(at 177.8 33.02 0)
 			(effects
 				(font
@@
 		)
 		(property "Sim.Device" "D"
-			(at 172.72 27.94 0)
+			(at 177.8 33.02 0)
 			(effects
 				(font
@@
 		)
 		(property "Sim.Pins" "1=K 2=A"
-			(at 172.72 27.94 0)
+			(at 177.8 33.02 0)
 			(effects
 				(font
